File: closed-loop-adapter/closed-loop-adapter/closed-loop-adapter.kicad_pcb (KiCad board)
At the start: 2 copper layers, 15.2 x 20.3 mm, 3 parts, among them J1 Conn_01x08_Pin, J2 Conn_01x08_Pin, J3 Conn_01x02_Pin

Commit message: feat: rework closed loop adapter
Parts:
- moved J3 4.57 mm to (109.4, 99.5), turned to 180 degrees
Connections:
- J1 pad 6: Net-(J1-Pin_6) -> unconnected-(J1-Pin_6-Pad6)
- J2 pad 2: unconnected-(J2-Pin_2-Pad2) -> Net-(J2-Pin_2)
- J2 pad 3: Net-(J1-Pin_8) -> Net-(J2-Pin_2)
- J2 pad 4: Net-(J1-Pin_7) -> Net-(J1-Pin_8)
- J2 pad 5: Net-(J1-Pin_6) -> Net-(J1-Pin_7)
Routing:
- net Net-(J1-Pin_1): track 16.2 -> 35.0 mm
- net Net-(J1-Pin_6): track 17.0 -> 0.00 mm
- net Net-(J1-Pin_8): track 22.1 -> 16.0 mm
- net Net-(J2-Pin_2): track 0.00 -> 2.54 mm
- net Net-(J1-Pin_7): track 19.3 -> 18.6 mm
- net Net-(J2-Pin_8): track 9.64 -> 10.2 mm
- net GND: vias 18 -> 16
Other:
- board text added: "B1 | EN B2 | CLK A2 | DIR A1 | VCC"
- board text added: "CLK"
- board text added: "DIR"
- board text added: "EN"
- board text added: "GND"
- board text added: "VCC"
- board text added: "VIN"
