File: closed-loop-adapter/closed-loop-adapter/closed-loop-adapter.kicad_sch (KiCad schematic)
At the start: 3 parts, among them J1 Conn_01x08_Pin, J2 Conn_01x08_Pin, J3 Conn_01x02_Pin

Commit message: feat: rework closed loop adapter
Connections:
- net at J2.2 (Pin_2): now also J2.3 (Pin_3)
- net at J1.8 (Pin_8): now also J2.4 (Pin_4); no longer J2.3 (Pin_3)
- net at J1.7 (Pin_7): now also J2.5 (Pin_5); no longer J2.4 (Pin_4)
- net at J1.6 (Pin_6): no longer J2.5 (Pin_5)
Changed lines of the file:
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@@
-	)
-	(no_connect
-		(at 119.38 91.44)
 	)
 	(no_connect
@@
 		(at 87.63 78.74)
 	)
+	(no_connect
+		(at 87.63 88.9)
+	)
 	(wire
 		(pts
-			(xy 93.98 83.82) (xy 119.38 83.82)
+			(xy 100.33 86.36) (xy 119.38 86.36)
 		)
 		(stroke
@@
 	(wire
 		(pts
-			(xy 93.98 88.9) (xy 93.98 83.82)
+			(xy 119.38 88.9) (xy 119.38 91.44)
 		)
 		(stroke
@@
 	(wire
 		(pts
-			(xy 87.63 91.44) (xy 96.52 91.44)
-		)
-		(stroke
-			(width 0)
-			(type default)
-		)
-	)
-	(wire
-		(pts
-			(xy 87.63 88.9) (xy 93.98 88.9)
+			(xy 97.79 83.82) (xy 119.38 83.82)
 		)
 		(stroke
@@
 	(wire
 		(pts
-			(xy 96.52 91.44) (xy 96.52 86.36)
+			(xy 87.63 93.98) (xy 100.33 93.98)
 		)
 		(stroke
@@
 	(wire
 		(pts
-			(xy 87.63 93.98) (xy 99.06 93.98)
+			(xy 100.33 93.98) (xy 100.33 86.36)
 		)
 		(stroke
@@
 	(wire
 		(pts
-			(xy 96.52 86.36) (xy 119.38 86.36)
+			(xy 87.63 91.44) (xy 97.79 91.44)
 		)
 		(stroke
@@
 	(wire
 		(pts
-			(xy 99.06 93.98) (xy 99.06 88.9)
+			(xy 97.79 91.44) (xy 97.79 83.82)
 		)
 		(stroke
@@
 		)
 		(stroke
-			(width 0)
-			(type default)
-		)
-	)
-	(wire
-		(pts
-			(xy 99.06 88.9) (xy 119.38 88.9)
-		)
-		(stroke
